File: ESP32V1 based led+button.sch (EAGLE design)
At the start: 11 parts

Commit message: edited files
Parts:
- added R4, R5, R6, R7, R8, R9: 330, SparkFun-Resistors:330OHM-HORIZ-1/10W-5%
Connections:
- new net B1: R5.2, U$2.IO19
- new net B2: R8.2, U$2.IO32
- new net G1: R4.2, U$2.IO18
- new net G2: R9.2, U$2.IO33
- new net N$10: D2.RED, R7.1
- new net N$17: D2.GRN, R9.1
- new net R1: R6.2, U$2.IO5
- new net R2: R7.2, U$2.IO25
- new net RX0: J1.3, U$2.IO3
- new net RX2: J2.3, U$2.IO16
- new net TX0: J1.2, U$2.IO1
- new net TX2: J2.2, U$2.IO17
- net GND: no longer U$2.GND1
- net N$5: now also D1.GRN, R4.1; no longer J1.3
- net N$6: now also D1.BLU, R5.1; no longer J1.2
- net N$7: now also D1.RED, R6.1; no longer J2.2
- net N$8: now also D2.BLU, R8.1; no longer J2.3
Other:
- moved on the sheet: D2
