File: PCB_Zero_prototype/ESP32V1 based led+button.brd (EAGLE design)
At the start: 72.1 x 50.5 mm, 17 parts

Commit message: added
Parts:
- moved JUMPER_1 4.89 mm to (56.1, 54.6), turned to 0 degrees
- moved JUMPER_2 4.23 mm to (61.7, 54.6)
- moved R2 2.09 mm to (38.6, 54.6), turned to 270 degrees
- moved R1 2.05 mm to (22.9, 54.9), turned to 270 degrees
Routing:
- net GND: track 115.4 -> 122.8 mm, vias 0 -> 2
- net N$3: track 42.4 -> 48.8 mm
- net N$16: track 49.0 -> 53.7 mm
- net RX0: track 25.3 -> 29.1 mm
- net N$6: track 25.9 -> 29.3 mm
- net TX0: track 21.3 -> 24.6 mm
- net N$9: track 55.8 -> 54.2 mm
- net +3V3: track 145.1 -> 143.7 mm
- net TX2: track 41.6 -> 43.0 mm
- net N$15: track 27.7 -> 28.9 mm
- net N$1: track 35.8 -> 34.6 mm
- net VCC: track 72.2 -> 73.1 mm
- net RX2: track 37.5 -> 38.4 mm
- net B1: track 5.86 -> 5.26 mm
- net G1: track 6.13 -> 5.54 mm
Other:
- board size 72.1 x 50.5 mm -> 74.2 x 56.9 mm
- board text added: "Zero Prototype Qu"
